File: pcb/indoor_weather_monitor.kicad_sch (KiCad schematic)
At the start: 3 parts, among them U1 DOIT-ESP32-DEVKIT-V1, U2 4.0inch_SPI_MSP4021, U2_BME280 module_bme280

Commit message: working on separate current conditions display
Connections:
- net at U1.19 (3V3), U2_BME280.1 (VCC): no longer U2.8 (LED)
- net at U2.5 (DC/RS): now also U1.9 (GPIO26_ADC2-CH9_DAC2_RTC-GPIO7); no longer U1.35 (GPIO22_I2C-SCL)
- net at U1.26 (GPIO4_ADC2-CH0_RTC-GPIO10): now also U2.8 (LED)
Changed lines of the file:
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@@
   (junction (at 162.56 76.835) (diameter 0) (color 0 0 0 0)
   )
-  (junction (at 167.64 84.455) (diameter 0) (color 0 0 0 0)
-  )
   (wire (pts (xy 78.74 53.975) (xy 91.44 53.975))
     (stroke (width 0) (type default) (color 0 0 0 0))
@@
     (stroke (width 0) (type default) (color 0 0 0 0))
   )
+  (wire (pts (xy 138.43 66.675) (xy 167.64 66.675))
+    (stroke (width 0) (type default) (color 0 0 0 0))
+  )
   (wire (pts (xy 91.44 56.515) (xy 80.645 56.515))
     (stroke (width 0) (type default) (color 0 0 0 0))
@@
     (stroke (width 0) (type default) (color 0 0 0 0))
   )
-  (wire (pts (xy 144.78 43.815) (xy 138.43 43.815))
-    (stroke (width 0) (type default) (color 0 0 0 0))
-  )
   (wire (pts (xy 155.575 40.64) (xy 155.575 42.545))
     (stroke (width 0) (type default) (color 0 0 0 0))
@@
     (stroke (width 0) (type default) (color 0 0 0 0))
   )
+  (wire (pts (xy 172.085 48.26) (xy 172.085 94.615))
+    (stroke (width 0) (type default) (color 0 0 0 0))
+  )
   (wire (pts (xy 144.78 53.975) (xy 144.78 58.42))
     (stroke (width 0) (type default) (color 0 0 0 0))
@@
     (stroke (width 0) (type default) (color 0 0 0 0))
   )
+  (wire (pts (xy 172.085 94.615) (xy 81.915 94.615))
+    (stroke (width 0) (type default) (color 0 0 0 0))
+  )
   (wire (pts (xy 179.07 58.42) (xy 144.78 58.42))
     (stroke (width 0) (type default) (color 0 0 0 0))
@@
     (stroke (width 0) (type default) (color 0 0 0 0))
   )
-  (wire (pts (xy 179.07 48.26) (xy 144.78 48.26))
-    (stroke (width 0) (type default) (color 0 0 0 0))
-  )
   (wire (pts (xy 144.78 58.42) (xy 144.78 88.265))
     (stroke (width 0) (type default) (color 0 0 0 0))
@@
     (stroke (width 0) (type default) (color 0 0 0 0))
   )
+  (wire (pts (xy 81.915 94.615) (xy 81.915 61.595))
+    (stroke (width 0) (type default) (color 0 0 0 0))
+  )
   (wire (pts (xy 141.605 59.055) (xy 141.605 78.74))
     (stroke (width 0) (type default) (color 0 0 0 0))
@@
     (stroke (width 0) (type default) (color 0 0 0 0))
   )
+  (wire (pts (xy 167.64 66.675) (xy 167.64 55.88))
+    (stroke (width 0) (type default) (color 0 0 0 0))
+  )
   (wire (pts (xy 78.74 100.33) (xy 78.74 53.975))
     (stroke (width 0) (type default) (color 0 0 0 0))
@@
     (stroke (width 0) (type default) (color 0 0 0 0))
   )
+  (wire (pts (xy 81.915 61.595) (xy 91.44 61.595))
+    (stroke (width 0) (type default) (color 0 0 0 0))
+  )
   (wire (pts (xy 179.07 45.72) (xy 160.02 45.72))
     (stroke (width 0) (type default) (color 0 0 0 0))
@@
     (stroke (width 0) (type default) (color 0 0 0 0))
   )
+  (wire (pts (xy 179.07 48.26) (xy 172.085 48.26))
+    (stroke (width 0) (type default) (color 0 0 0 0))
+  )
   (wire (pts (xy 151.13 41.275) (xy 138.43 41.275))
     (stroke (width 0) (type default) (color 0 0 0 0))
@@
     (stroke (width 0) (type default) (color 0 0 0 0))
   )
-  (wire (pts (xy 144.78 48.26) (xy 144.78 43.815))
-    (stroke (width 0) (type default) (color 0 0 0 0))
-  )
   (wire (pts (xy 155.575 40.64) (xy 179.07 40.64))
     (stroke (width 0) (type default) (color 0 0 0 0))
   )
-  (wire (pts (xy 167.64 55.88) (xy 167.64 84.455))
-    (stroke (width 0) (type default) (color 0 0 0 0))
-  )

Commit message: tooling around with placement
Parts:
- added U3_BH1750: module_bh1750, usini_sensors:module_bh1750, symbol usini_sensors:module_bh1750
Connections:
- net GND: now also U3_BH1750.4 (GND)
- net at U1.30 (GPIO18_VSPI-CLK), U2.18 (SD_SCK), U2.7 (SCK)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: now also U1.35 (GPIO22_I2C-SCL), U3_BH1750.3 (SCL)
- net at U1.18 (VIN), U2.1 (VCC): now also U3_BH1750.5 (VCC)
- net at U1.32 (GPIO21_I2C-SDA): now also U3_BH1750.2 (SDA)
Changed lines of the file:
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@@
 (kicad_sch (version 20211123) (generator eeschema)
   (paper "A4")
+  (junction (at 147.32 56.515) (diameter 0) (color 0 0 0 0)
+  )
   (junction (at 151.13 90.805) (diameter 0) (color 0 0 0 0)
   )
@@
   (junction (at 144.78 88.265) (diameter 0) (color 0 0 0 0)
   )
+  (junction (at 147.32 53.34) (diameter 0) (color 0 0 0 0)
+  )
   (junction (at 162.56 76.835) (diameter 0) (color 0 0 0 0)
   )
+  (junction (at 111.76 93.345) (diameter 0) (color 0 0 0 0)
+  )
   (wire (pts (xy 78.74 53.975) (xy 91.44 53.975))
     (stroke (width 0) (type default) (color 0 0 0 0))
@@
     (stroke (width 0) (type default) (color 0 0 0 0))
   )
+  (wire (pts (xy 78.74 134.62) (xy 147.32 134.62))
+    (stroke (width 0) (type default) (color 0 0 0 0))
+  )
   (wire (pts (xy 209.55 38.1) (xy 201.93 38.1))
     (stroke (width 0) (type default) (color 0 0 0 0))
@@
     (stroke (width 0) (type default) (color 0 0 0 0))
   )
+  (wire (pts (xy 147.32 43.815) (xy 138.43 43.815))
+    (stroke (width 0) (type default) (color 0 0 0 0))
+  )
   (wire (pts (xy 155.575 40.64) (xy 155.575 42.545))
     (stroke (width 0) (type default) (color 0 0 0 0))
@@
     (stroke (width 0) (type default) (color 0 0 0 0))
   )
+  (wire (pts (xy 111.76 130.175) (xy 111.76 93.345))
+    (stroke (width 0) (type default) (color 0 0 0 0))
+  )
   (wire (pts (xy 91.44 84.455) (xy 88.9 84.455))
     (stroke (width 0) (type default) (color 0 0 0 0))
@@
     (stroke (width 0) (type default) (color 0 0 0 0))
   )
+  (wire (pts (xy 87.63 125.095) (xy 87.63 130.175))
+    (stroke (width 0) (type default) (color 0 0 0 0))
+  )
   (wire (pts (xy 144.78 53.975) (xy 138.43 53.975))
     (stroke (width 0) (type default) (color 0 0 0 0))
   )
+  (wire (pts (xy 78.74 120.015) (xy 78.74 134.62))
+    (stroke (width 0) (type default) (color 0 0 0 0))
+  )
   (wire (pts (xy 167.64 84.455) (xy 167.64 114.935))
     (stroke (width 0) (type default) (color 0 0 0 0))
@@
     (stroke (width 0) (type default) (color 0 0 0 0))
   )
+  (wire (pts (xy 87.63 117.475) (xy 83.185 117.475))
+    (stroke (width 0) (type default) (color 0 0 0 0))
+  )
   (wire (pts (xy 144.78 58.42) (xy 144.78 88.265))
     (stroke (width 0) (type default) (color 0 0 0 0))
@@
     (stroke (width 0) (type default) (color 0 0 0 0))
   )
+  (wire (pts (xy 87.63 130.175) (xy 111.76 130.175))
+    (stroke (width 0) (type default) (color 0 0 0 0))
+  )
   (wire (pts (xy 151.13 50.8) (xy 151.13 41.275))
     (stroke (width 0) (type default) (color 0 0 0 0))
   )
-  (wire (pts (xy 88.9 93.345) (xy 153.035 93.345))
+  (wire (pts (xy 88.9 93.345) (xy 111.76 93.345))
     (stroke (width 0) (type default) (color 0 0 0 0))
   )
@@
     (stroke (width 0) (type default) (color 0 0 0 0))
   )
+  (wire (pts (xy 138.43 51.435) (xy 142.24 51.435))
+    (stroke (width 0) (type default) (color 0 0 0 0))
+  )
   (wire (pts (xy 173.355 120.015) (xy 162.56 120.015))
     (stroke (width 0) (type default) (color 0 0 0 0))
   )
+  (wire (pts (xy 111.76 93.345) (xy 153.035 93.345))
+    (stroke (width 0) (type default) (color 0 0 0 0))
+  )
   (wire (pts (xy 179.07 55.88) (xy 167.64 55.88))
     (stroke (width 0) (type default) (color 0 0 0 0))
@@
     (stroke (width 0) (type default) (color 0 0 0 0))
   )
+  (wire (pts (xy 87.63 120.015) (xy 78.74 120.015))
+    (stroke (width 0) (type default) (color 0 0 0 0))
+  )
   (wire (pts (xy 151.13 90.805) (xy 207.01 90.805))
     (stroke (width 0) (type default) (color 0 0 0 0))
@@
     (stroke (width 0) (type default) (color 0 0 0 0))
   )
+  (wire (pts (xy 142.24 106.045) (xy 142.24 51.435))
+    (stroke (width 0) (type default) (color 0 0 0 0))
+  )
   (wire (pts (xy 81.915 94.615) (xy 81.915 61.595))
     (stroke (width 0) (type default) (color 0 0 0 0))
@@
     (stroke (width 0) (type default) (color 0 0 0 0))
   )
+  (wire (pts (xy 83.185 117.475) (xy 83.185 106.045))
+    (stroke (width 0) (type default) (color 0 0 0 0))
+  )
   (wire (pts (xy 167.64 66.675) (xy 167.64 55.88))
     (stroke (width 0) (type default) (color 0 0 0 0))
@@
     (stroke (width 0) (type default) (color 0 0 0 0))
   )
+  (wire (pts (xy 147.32 43.815) (xy 147.32 53.34))
+    (stroke (width 0) (type default) (color 0 0 0 0))
+  )
+  (wire (pts (xy 167.64 114.935) (xy 173.355 114.935))
+    (stroke (width 0) (type default) (color 0 0 0 0))
+  )
+  (wire (pts (xy 80.645 97.155) (xy 158.115 97.155))
+    (stroke (width 0) (type default) (color 0 0 0 0))
+  )
+  (wire (pts (xy 162.56 53.34) (xy 147.32 53.34))
+    (stroke (width 0) (type default) (color 0 0 0 0))
+  )
+  (wire (pts (xy 81.915 61.595) (xy 91.44 61.595))
+    (stroke (width 0) (type default) (color 0 0 0 0))
+  )
+  (wire (pts (xy 179.07 45.72) (xy 160.02 45.72))
+    (stroke (width 0) (type default) (color 0 0 0 0))
+  )
+  (wire (pts (xy 167.64 117.475) (xy 173.355 117.475))
+    (stroke (width 0) (type default) (color 0 0 0 0))
+  )
+  (wire (pts (xy 179.07 50.8) (xy 151.13 50.8))
+    (stroke (width 0) (type default) (color 0 0 0 0))
+  )
+  (wire (pts (xy 88.9 84.455) (xy 88.9 93.345))
+    (stroke (width 0) (type default) (color 0 0 0 0))
+  )
+  (wire (pts (xy 83.82 81.915) (xy 83.82 88.265))
+    (stroke (width 0) (type default) (color 0 0 0 0))
+  )
+  (wire (pts (xy 81.28 122.555) (xy 81.28 124.46))
+    (stroke (width 0) (type default) (color 0 0 0 0))
+  )
+  (wire (pts (xy 146.05 71.755) (xy 138.43 71.755))
+    (stroke (width 0) (type default) (color 0 0 0 0))
+  )
+  (wire (pts (xy 207.01 41.275) (xy 201.93 41.275))
+    (stroke (width 0) (type default) (color 0 0 0 0))
+  )
+  (wire (pts (xy 173.355 122.555) (xy 151.13 122.555))
+    (stroke (width 0) (type default) (color 0 0 0 0))
+  )
   (wire (pts (xy 147.32 53.34) (xy 147.32 56.515))
     (stroke (width 0) (type default) (color 0 0 0 0))
   )
-  (wire (pts (xy 167.64 114.935) (xy 173.355 114.935))
-    (stroke (width 0) (type default) (color 0 0 0 0))
-  )
-  (wire (pts (xy 80.645 97.155) (xy 158.115 97.155))
-    (stroke (width 0) (type default) (color 0 0 0 0))
-  )
-  (wire (pts (xy 162.56 53.34) (xy 147.32 53.34))
-    (stroke (width 0) (type default) (color 0 0 0 0))
-  )
-  (wire (pts (xy 81.915 61.595) (xy 91.44 61.595))
-    (stroke (width 0) (type default) (color 0 0 0 0))
-  )
-  (wire (pts (xy 179.07 45.72) (xy 160.02 45.72))
-    (stroke (width 0) (type default) (color 0 0 0 0))
-  )
-  (wire (pts (xy 167.64 117.475) (xy 173.355 117.475))
-    (stroke (width 0) (type default) (color 0 0 0 0))
-  )
-  (wire (pts (xy 179.07 50.8) (xy 151.13 50.8))
-    (stroke (width 0) (type default) (color 0 0 0 0))
-  )
-  (wire (pts (xy 88.9 84.455) (xy 88.9 93.345))
-    (stroke (width 0) (type default) (color 0 0 0 0))
-  )
-  (wire (pts (xy 83.82 81.915) (xy 83.82 88.265))
-    (stroke (width 0) (type default) (color 0 0 0 0))
-  )
-  (wire (pts (xy 146.05 71.755) (xy 138.43 71.755))
-    (stroke (width 0) (type default) (color 0 0 0 0))
-  )
-  (wire (pts (xy 207.01 41.275) (xy 201.93 41.275))
-    (stroke (width 0) (type default) (color 0 0 0 0))
-  )
-  (wire (pts (xy 173.355 122.555) (xy 151.13 122.555))
-    (stroke (width 0) (type default) (color 0 0 0 0))
-  )
   (wire (pts (xy 146.05 125.095) (xy 146.05 71.755))
     (stroke (width 0) (type default) (color 0 0 0 0))
@@
   )
   (wire (pts (xy 151.13 41.275) (xy 138.43 41.275))
+    (stroke (width 0) (type default) (color 0 0 0 0))
+  )
+  (wire (pts (xy 83.185 106.045) (xy 142.24 106.045))
+    (stroke (width 0) (type default) (color 0 0 0 0))
+  )
+  (wire (pts (xy 147.32 56.515) (xy 147.32 134.62))
+    (stroke (width 0) (type default) (color 0 0 0 0))
+  )
+  (wire (pts (xy 87.63 122.555) (xy 81.28 122.555))
     (stroke (width 0) (type default) (color 0 0 0 0))
   )
@@
     (pin "9")
   )
+  (symbol (lib_id "usini_sensors:module_bh1750") (at 87.63 122.555 0) (unit 1)
+    (in_bom yes) (on_board yes)
+    (property "Reference" "U3_BH1750" (id 0) (at 91.44 112.395 0))
+    (property "Value" "module_bh1750" (id 1) (at 97.79 127.635 0))
+    (property "Footprint" "usini_sensors:module_bh1750" (id 2) (at 97.79 130.175 0)
+      (effects (font (size 1.27 1.27)) hide)
+    )
+    (property "Datasheet" "" (id 3) (at 87.63 122.555 0)
+      (effects (font (size 1.27 1.27)) hide)
+    )
+    (pin "1")
+    (pin "2")
+    (pin "3")
+    (pin "4")
+    (pin "5")
+  )
   (symbol (lib_id "power:GND") (at 167.64 117.475 0) (unit 1)
     (in_bom yes) (on_board yes)
@@
     )
     (property "Datasheet" "" (id 3) (at 167.64 117.475 0)
+      (effects (font (size 1.27 1.27)) hide)
+    )
+    (pin "1")
+  )
+  (symbol (lib_id "power:GND") (at 81.28 124.46 0) (unit 1)
+    (in_bom yes) (on_board yes)
+    (property "Reference" "#PWR0104" (id 0) (at 81.28 130.81 0)
+      (effects (font (size 1.27 1.27)) hide)
+    )
+    (property "Value" "GND" (id 1) (at 81.28 128.27 0))
+    (property "Footprint" "" (id 2) (at 81.28 124.46 0)
+      (effects (font (size 1.27 1.27)) hide)
+    )
+    (property "Datasheet" "" (id 3) (at 81.28 124.46 0)
       (effects (font (size 1.27 1.27)) hide)
     )
@@
       (reference "#PWR0103") (unit 1) (value "GND") (footprint "")
     )
+    (path "/7e0a94a5-71e1-4db6-a3c9-ed35b8d6c216"
+      (reference "#PWR0104") (unit 1) (value "GND") (footprint "")
+    )
     (path "/a95b6208-cd25-486f-8a35-f7d7b1426174"
       (reference "U1") (unit 1) (value "DOIT-ESP32-DEVKIT-V1") (footprint "esp32:MODULE_ESP32_DEVKIT_V1")
@@
       (reference "U2_BME280") (unit 1) (value "module_bme280") (footprint "usini_sensors:module_bme280")
     )
-  )
+    (path "/5e27c7e3-130d-477a-b693-9d7d6d05e3e3"
+      (reference "U3_BH1750") (unit 1) (value "module_bh1750") (footprint "usini_sensors:module_bh1750")
+    )
+  )
